Commit message: deptHoled mode fixed

File: src/robot_description/urdf/ardusub.urdf.xacro (robot description, xacro)
@@ -19,11 +19,14 @@
       <connectionTimeoutMaxCount>5</connectionTimeoutMaxCount>
       <!--
-        ArduSub Motor 1 is front-right.  The CAD / URDF link names are
-        mirrored relative to the ArduSub mixer, so pairwise routing is used:
-        it keeps surge correct while restoring sway and yaw signs.
+        ArduSub VECTORED mixer (FRAME_CONFIG=1), in physical vehicle order.
+        The force axes calculated from the URDF joint poses are:
+          M1=t4 front-right, M2=t3 front-left,
+          M3=t2 rear-right,  M4=t1 rear-left.
+        Negative multipliers map ArduSub's surge / sway / yaw allocation to
+        the physical forward direction of the visual model.
       -->
       <control channel="0">
         <type>COMMAND</type>
-        <jointName>t2_joint</jointName>
+        <jointName>t4_joint</jointName>
         <offset>-0.5</offset>
         <!-- Positive ArduSub forward command must produce Gazebo forward thrust. -->
@@ -31,8 +34,28 @@
         <servo_min>1100</servo_min>
         <servo_max>1900</servo_max>
-        <cmd_topic>/model/robot_description/joint/t2_joint/cmd_thrust</cmd_topic>
+        <cmd_topic>/model/robot_description/joint/t4_joint/cmd_thrust</cmd_topic>
       </control>
       <!-- ArduSub Motor 2 is front-left. -->
       <control channel="1">
+        <type>COMMAND</type>
+        <jointName>t3_joint</jointName>
+        <offset>-0.5</offset>
+        <multiplier>-103.0</multiplier>
+        <servo_min>1100</servo_min>
+        <servo_max>1900</servo_max>
+        <cmd_topic>/model/robot_description/joint/t3_joint/cmd_thrust</cmd_topic>
+      </control>
+      <!-- ArduSub Motor 3 is rear-right. -->
+      <control channel="2">
+        <type>COMMAND</type>
+        <jointName>t2_joint</jointName>
+        <offset>-0.5</offset>
+        <multiplier>-103.0</multiplier>
+        <servo_min>1100</servo_min>
+        <servo_max>1900</servo_max>
+        <cmd_topic>/model/robot_description/joint/t2_joint/cmd_thrust</cmd_topic>
+      </control>
+      <!-- ArduSub Motor 4 is rear-left. -->
+      <control channel="3">
         <type>COMMAND</type>
         <jointName>t1_joint</jointName>
@@ -43,40 +66,22 @@
         <cmd_topic>/model/robot_description/joint/t1_joint/cmd_thrust</cmd_topic>
       </control>
-      <!-- ArduSub Motor 3 is rear-right. -->
-      <control channel="2">
+      <!-- ArduSub Motor 5: vertical left.  Negative gain maps ArduSub heave
+           commands to the physical thrust direction of this Gazebo joint. -->
+      <control channel="4">
         <type>COMMAND</type>
-        <jointName>t4_joint</jointName>
+        <jointName>t5_joint</jointName>
         <offset>-0.5</offset>
         <multiplier>-103.0</multiplier>
         <servo_min>1100</servo_min>
         <servo_max>1900</servo_max>
-        <cmd_topic>/model/robot_description/joint/t4_joint/cmd_thrust</cmd_topic>
-      </control>
-      <!-- ArduSub Motor 4 is rear-left. -->
-      <control channel="3">
-        <type>COMMAND</type>
-        <jointName>t3_joint</jointName>
-        <offset>-0.5</offset>
-        <multiplier>-103.0</multiplier>
-        <servo_min>1100</servo_min>
-        <servo_max>1900</servo_max>
-        <cmd_topic>/model/robot_description/joint/t3_joint/cmd_thrust</cmd_topic>
-      </control>
-      <!-- ArduSub Motor 5: vertical left.  Positive gain corrects the observed inverted heave response. -->
-      <control channel="4">
-        <type>COMMAND</type>
-        <jointName>t5_joint</jointName>
-        <offset>-0.5</offset>
-        <multiplier>103.0</multiplier>
-        <servo_min>1100</servo_min>
-        <servo_max>1900</servo_max>
         <cmd_topic>/model/robot_description/joint/t5_joint/cmd_thrust</cmd_topic>
       </control>
-      <!-- ArduSub Motor 6: vertical right.  Positive gain corrects the observed inverted heave response. -->
+      <!-- ArduSub Motor 6: vertical right.  Keep the same heave polarity as
+           Motor 5 so collective vertical commands do not invert. -->
       <control channel="5">
         <type>COMMAND</type>
         <jointName>t6_joint</jointName>
         <offset>-0.5</offset>
-        <multiplier>103.0</multiplier>
+        <multiplier>-103.0</multiplier>
         <servo_min>1100</servo_min>
         <servo_max>1900</servo_max>

File: src/robot_description/urdf/robot_description.urdf (robot description, URDF)
Before this commit: robot robot_description, 11 links, 10 joints
Links:
- link center_body_link: geometry collision box size=0.30 0.1540825943 0.45; visual mesh filename=package://robot_description/meshes/center_body_link.STL
Joints:
- joint imu_joint: origin xyz=0 0 0 rpy=0 0 0 -> xyz=0 0 0 rpy=3.141592653589793 0 0
- joint t1_joint: origin xyz=0.13838 -0.054 0.1764 rpy=0 0.7854 -3.1416 -> xyz=0.13838 -0.054 0.1764 rpy=0 0.7853981633974483 -3.141592653589793
- joint t2_joint: origin xyz=-0.13844 -0.054 0.1764 rpy=0 0.7854 0 -> xyz=-0.13844 -0.054 0.1764 rpy=0 0.7853981633974483 0
- joint t3_joint: origin xyz=0.13838 -0.054 -0.13678 rpy=3.1416 0.7854 0 -> xyz=0.13838 -0.054 -0.13678 rpy=3.141592653589793 0.7853981633974483 0
- joint t4_joint: origin xyz=-0.13844 -0.054 -0.13678 rpy=3.1416 -0.7854 0 -> xyz=-0.13844 -0.054 -0.13678 rpy=3.141592653589793 -0.7853981633974483 0
- joint t5_joint: origin xyz=0.16097 0.053527 0.01981 rpy=-1.5708 -0.0014872 0 -> xyz=0.16097 0.053527 0.01981 rpy=-1.5707963267948966 0 0
- joint t6_joint: origin xyz=-0.16103 0.053527 0.01981 rpy=-1.5708 -0.0014872 0 -> xyz=-0.16103 0.053527 0.01981 rpy=-1.5707963267948966 0 0

Commit message: Sync complete workspace with simulation, GUI, and assets

File: src/robot_description/urdf/ardusub.urdf.xacro (robot description, xacro)
@@ -1,32 +1,27 @@
 <?xml version="1.0" encoding="utf-8"?>
 <robot xmlns:xacro="http://www.ros.org/wiki/xacro">
+  <xacro:arg name="sitl_port_in" default="9002" />
+  <xacro:arg name="sitl_port_out" default="9003" />
   <!-- ================= ARDUPILOT SITL PLUGIN ================= -->
   <gazebo>
     <plugin filename="libArduPilotPlugin.so" name="gz::sim::v8::systems::ArduPilotPlugin">
       <fdm_addr>127.0.0.1</fdm_addr>
-      <fdm_port_in>9002</fdm_port_in>
-      <fdm_port_out>9003</fdm_port_out>
-      <!--
-        base_link follows ROS REP-103 (X forward, Y left, Z up).  ArduPilot
-        consumes body FRD and world NED.  A 180 degree roll is the required
-        FLU -> FRD conversion; a pitch rotation reverses the vehicle's forward
-        axis and was the cause of reversed manual motion.
-      -->
-      <modelXYZToAirplaneXForwardZDown>0 0 0 3.141593 0 0</modelXYZToAirplaneXForwardZDown>
+      <fdm_port_in>$(arg sitl_port_in)</fdm_port_in>
+      <fdm_port_out>$(arg sitl_port_out)</fdm_port_out>
+      <!-- The plugin reads pose from imu_link, already rotated FLU -> FRD.
+           Applying another 180-degree roll here would make the JSON attitude
+           disagree with the gyro and accelerometer. -->
+      <modelXYZToAirplaneXForwardZDown>0 0 0 0 0 0</modelXYZToAirplaneXForwardZDown>
       <!-- Gazebo world is ENU; ArduPilot world is NED. -->
       <gazeboXYZToNED>0 0 0 3.141593 0 1.570796</gazeboXYZToNED>
       <imuName>imu_sensor</imuName>
       <connectionTimeoutMaxCount>5</connectionTimeoutMaxCount>
-      <!--
-        ArduSub VECTORED mixer (FRAME_CONFIG=1), in physical vehicle order.
-        The force axes calculated from the URDF joint poses are:
-          M1=t4 front-right, M2=t3 front-left,
-          M3=t2 rear-right,  M4=t1 rear-left.
-        Negative multipliers map ArduSub's surge / sway / yaw allocation to
-        the physical forward direction of the visual model.
-      -->
+      <!-- Match ArduSub VECTORED allocation in the IMU FRD control frame:
+           M1=t3, M2=t4, M3=t1, M4=t2. Positive yaw must produce
+           negative Gazebo Z torque; swapping left/right produces feedback
+           with the wrong sign in STABILIZE and ALT_HOLD. -->
       <control channel="0">
         <type>COMMAND</type>
-        <jointName>t4_joint</jointName>
+        <jointName>t3_joint</jointName>
         <offset>-0.5</offset>
         <!-- Positive ArduSub forward command must produce Gazebo forward thrust. -->
@@ -34,18 +29,28 @@
         <servo_min>1100</servo_min>
         <servo_max>1900</servo_max>
-        <cmd_topic>/model/robot_description/joint/t4_joint/cmd_thrust</cmd_topic>
+        <cmd_topic>/model/robot_description/joint/t3_joint/cmd_thrust</cmd_topic>
       </control>
-      <!-- ArduSub Motor 2 is front-left. -->
+      <!-- ArduSub Motor 2 maps to t4. -->
       <control channel="1">
         <type>COMMAND</type>
-        <jointName>t3_joint</jointName>
+        <jointName>t4_joint</jointName>
         <offset>-0.5</offset>
         <multiplier>-103.0</multiplier>
         <servo_min>1100</servo_min>
         <servo_max>1900</servo_max>
-        <cmd_topic>/model/robot_description/joint/t3_joint/cmd_thrust</cmd_topic>
+        <cmd_topic>/model/robot_description/joint/t4_joint/cmd_thrust</cmd_topic>
       </control>
-      <!-- ArduSub Motor 3 is rear-right. -->
+      <!-- ArduSub Motor 3 maps to t1. -->
       <control channel="2">
+        <type>COMMAND</type>
+        <jointName>t1_joint</jointName>
+        <offset>-0.5</offset>
+        <multiplier>-103.0</multiplier>
+        <servo_min>1100</servo_min>
+        <servo_max>1900</servo_max>
+        <cmd_topic>/model/robot_description/joint/t1_joint/cmd_thrust</cmd_topic>
+      </control>
+      <!-- ArduSub Motor 4 maps to t2. -->
+      <control channel="3">
         <type>COMMAND</type>
         <jointName>t2_joint</jointName>
@@ -55,14 +60,4 @@
         <servo_max>1900</servo_max>
         <cmd_topic>/model/robot_description/joint/t2_joint/cmd_thrust</cmd_topic>
-      </control>
-      <!-- ArduSub Motor 4 is rear-left. -->
-      <control channel="3">
-        <type>COMMAND</type>
-        <jointName>t1_joint</jointName>
-        <offset>-0.5</offset>
-        <multiplier>-103.0</multiplier>
-        <servo_min>1100</servo_min>
-        <servo_max>1900</servo_max>
-        <cmd_topic>/model/robot_description/joint/t1_joint/cmd_thrust</cmd_topic>
       </control>
       <!-- ArduSub Motor 5: vertical left.  Negative gain maps ArduSub heave

File: src/robot_description/urdf/robot_description.urdf (robot description, URDF)
Before this commit: robot robot_description, 11 links, 10 joints
Links:
- removed link zed_link
- added link camera_dome_link; visual mesh filename=package://robot_description/meshes/appearance/dome.stl
- added link hydrodynamics_link, mass 0.001
- added link imu_ros_link
- added link rov_base_link
- link center_body_link: mass 20.277556 -> 20.226556000; geometry collision box size=0.01 0.012 0.113710000000; collision box size=0.01 0.012 0.113710000000
Joints:
- removed joint zed_joint
- added joint base_to_hydrodynamics: type fixed, parent base_link, child hydrodynamics_link, origin xyz=-0.019809801536 0.000030072765 -0.054000072766 rpy=0 0 0
- added joint base_to_rov_base: type fixed, parent base_link, child rov_base_link, origin xyz=0 0 0 rpy=0 0 3.141592653589793
- added joint center_body_to_camera_dome: type fixed, parent center_body_link, child camera_dome_link, origin xyz=0 0 0 rpy=0 0 0
- added joint rov_base_to_imu_ros: type fixed, parent rov_base_link, child imu_ros_link, origin xyz=0 0 0 rpy=0 0 0
- added joint zed2i_mount_joint: type fixed, parent rov_base_link, child zed2i_camera_link, origin xyz=0.186469391519 -0.000223754166 -0.0150005512922 rpy=0 0 0
